File: hardware/gbg_base_revb.sch (EAGLE design)
At the start: 15 parts, among them Q3 NTS4173, U1 AB0805, U2 USD-SOCKET, U3 LP2985AIM5-3.3

Commit message: new hardware, simple
Parts:
- removed C1: (no value), SparkFun-Passives:CAP1210
- removed JP1: (no value), SparkFun-Connectors:M02PTH
- removed Q3: NTS4173, nts4173p:NTS4173
- removed R1, R2: 4.7k, SparkFun-Resistors:RESISTOR0603
- removed R11: 220k, tiny_passives:R-EU0603
- removed R3: 1.5k, SparkFun-Resistors:RESISTOR0603
- removed U1: AB0805, AB08XX:AB0805
Connections:
- removed net N$1: C1.1, R3.1
- removed net N$5: R3.2, U1.VBAT
- removed net SD_VCC: Q3.D, U2.VCC
- net !SD_ENABLE: no longer Q3.G, R11.1
- net GND: no longer C1.2, JP1.1, U1.EXTI, U1.VSS, U1.WDI
- net I2C_SCL: no longer R2.1, U1.SCL
- net I2C_SDA: no longer R1.1, U1.SDA
- net VBAT: no longer JP1.2
- net VCC: now also U2.VCC; no longer Q3.S, R1.2, R11.2, R2.2, U1.VCC
Other:
- note removed: "Real Time Clock"
