File: hardware/gbgv02/boardPCBlayout2.brd (EAGLE design)
At the start: 56 x 51 mm, 44 parts, among them P1 0475890001, U1 MCP73833-CNI/UN, U2 USD-SOCKET, U3 BT832, U4 LP2985-30DBVRDBV5-L, U5 LSM9DS1

Commit message: polygons
Routing:
- net VCC: track 144.6 -> 6.02 mm, vias 8 -> 4
- added copper zone on layer 1, net GND
- added copper zone on layer 16, net VCC
